Commit message: modified:   source/wheel_leg_humanoid_lab/wheel_leg_humanoid_lab/assets/wheel_leg_humanoid_description/urdf/wheel_leg_humanoid.urdf 	modified:   source/wheel_leg_humanoid_lab/wheel_leg_humanoid_lab/assets/wheel_leg_humanoid_description/urdf/wheel_leg_humanoid/configuration/wheel_leg_humanoid_base.usd 	modified:   source/wheel_leg_humanoid_lab/wheel_leg_humanoid_lab/assets/wheel_leg_humanoid_description/urdf/wheel_leg_humanoid/configuration/wheel_leg_humanoid_physics.usd 	modified:   source/wheel_leg_humanoid_lab/wheel_leg_humanoid_lab/assets/wheel_leg_humanoid_description/urdf/wheel_leg_humanoid/configuration/wheel_leg_humanoid_robot.usd 	modified:   source/wheel_leg_humanoid_lab/wheel_leg_humanoid_lab/assets/wheel_leg_humanoid_description/urdf/wheel_leg_humanoid/wheel_leg_humanoid.usd 	deleted:    source/wheel_leg_humanoid_lab/wheel_leg_humanoid_lab/assets/wheel_leg_humanoid_description/usd/wheel_leg_humanoid/configuration/wheel_leg_humanoid_base.usd 	deleted:    source/wheel_leg_humanoid_lab/wheel_leg_humanoid_lab/assets/wheel_leg_humanoid_description/usd/wheel_leg_humanoid/configuration/wheel_leg_humanoid_physics.usd 	deleted:    source/wheel_leg_humanoid_lab/wheel_leg_humanoid_lab/assets/wheel_leg_humanoid_description/usd/wheel_leg_humanoid/configuration/wheel_leg_humanoid_robot.usd 	deleted:    source/wheel_leg_humanoid_lab/wheel_leg_humanoid_lab/assets/wheel_leg_humanoid_description/usd/wheel_leg_humanoid/configuration/wheel_leg_humanoid_sensor.usd 	deleted:    source/wheel_leg_humanoid_lab/wheel_leg_humanoid_lab/assets/wheel_leg_humanoid_description/usd/wheel_leg_humanoid/wheel_leg_humanoid.usd

File: source/wheel_leg_humanoid_lab/wheel_leg_humanoid_lab/assets/wheel_leg_humanoid_description/urdf/wheel_leg_humanoid.urdf (robot description, URDF)
Before this commit: robot wheel_leg_humanoid, 20 links, 19 joints
Links:
- link left_ankle_2: mass 4.561092579439662 -> 1.55786
- link left_thigh: mass 11.979286445373326 -> 5.25364
- link left_wheel: mass 6.388973210532128 -> 1.0
- link right_ankle_2: mass 4.7664343049317335 -> 1.55786
- link right_foot_wheel_L: mass 0.23598528385264425 -> 0.235985283852645
- link right_thigh: mass 11.981536969926172 -> 5.25364
- link right_wheel: mass 6.388989701638672 -> 1.0
Joints:
- joint left_ankle_1: limit lower=-0.52 upper=0.87 effort=24.8 velocity=10.8 -> lower=-0.610865 upper=0.610865 effort=24.8 velocity=10.8
- joint left_ankle_2: limit lower=-0.523599 upper=0.523599 effort=24.8 velocity=10.8 -> lower=-0.209439 upper=0.209439 effort=24.8 velocity=10.8
- joint left_calf: limit lower=-0.26 upper=2.05 effort=120 velocity=5.02 -> lower=0.0 upper=2.094395 effort=120 velocity=5.02
- joint left_pelvis_1: limit lower=-2.094395 upper=2.094395 effort=120 velocity=5.02 -> lower=-1.57 upper=1.57 effort=120 velocity=5.02
- joint left_pelvis_2: limit lower=-0.174533 upper=0.43 effort=120 velocity=5.02 -> lower=-0.261799 upper=1.57 effort=120 velocity=5.02
- joint left_thigh: limit lower=-0.43 upper=0.43 effort=120 velocity=5.02 -> lower=-1.57 upper=1.57 effort=120 velocity=5.02
- joint right_ankle_1: limit lower=-0.87 upper=0.52 effort=24.8 velocity=10.8 -> lower=-0.610865 upper=0.610865 effort=24.8 velocity=10.8
- joint right_ankle_2: limit lower=-0.523599 upper=0.523599 effort=24.8 velocity=10.8 -> lower=-0.209439 upper=0.209439 effort=24.8 velocity=10.8
- joint right_calf: limit lower=-2.05 upper=0.26 effort=120 velocity=5.02 -> lower=-2.094395 upper=0.0 effort=120 velocity=5.02
- joint right_pelvis_1: limit lower=-2.094395 upper=2.094395 effort=120 velocity=5.02 -> lower=-1.57 upper=1.57 effort=120 velocity=5.02
- joint right_pelvis_2: limit lower=-0.43 upper=0.174533 effort=120 velocity=5.02 -> lower=-1.57 upper=0.261799 effort=120 velocity=5.02
- joint right_thigh: limit lower=-0.43 upper=0.43 effort=120 velocity=5.02 -> lower=-1.57 upper=1.57 effort=120 velocity=5.02

Commit message: modified:   source/wheel_leg_humanoid_lab/wheel_leg_humanoid_lab/assets/utils/get_com_from_urdf.py 	modified:   source/wheel_leg_humanoid_lab/wheel_leg_humanoid_lab/assets/wheel_leg_humanoid.py 	modified:   source/wheel_leg_humanoid_lab/wheel_leg_humanoid_lab/assets/wheel_leg_humanoid_description/urdf/wheel_leg_humanoid.urdf 	modified:   source/wheel_leg_humanoid_lab/wheel_leg_humanoid_lab/assets/wheel_leg_humanoid_description/urdf/wheel_leg_humanoid/configuration/wheel_leg_humanoid_base.usd 	modified:   source/wheel_leg_humanoid_lab/wheel_leg_humanoid_lab/assets/wheel_leg_humanoid_description/urdf/wheel_leg_humanoid/configuration/wheel_leg_humanoid_physics.usd 	modified:   source/wheel_leg_humanoid_lab/wheel_leg_humanoid_lab/assets/wheel_leg_humanoid_description/urdf/wheel_leg_humanoid/wheel_leg_humanoid.usd 	modified:   source/wheel_leg_humanoid_lab/wheel_leg_humanoid_lab/tasks/manager_based/wheel_leg_humanoid/velocity/config/drving/rough_env_cfg.py 	modified:   source/wheel_leg_humanoid_lab/wheel_leg_humanoid_lab/tasks/manager_based/wheel_leg_humanoid/velocity/config/walking/__pycache__/rough_env_cfg.cpython-311.pyc 	modified:   source/wheel_leg_humanoid_lab/wheel_leg_humanoid_lab/tasks/manager_based/wheel_leg_humanoid/velocity/config/walking/rough_env_cfg.py

File: source/wheel_leg_humanoid_lab/wheel_leg_humanoid_lab/assets/wheel_leg_humanoid_description/urdf/wheel_leg_humanoid.urdf (robot description, URDF)
Before this commit: robot wheel_leg_humanoid, 20 links, 19 joints
Joints:
- joint right_calf: limit lower=-2.094395 upper=0.0 effort=120 velocity=5.02 -> lower=0.0 upper=2.094395 effort=120 velocity=5.02

Commit message: modified:   source/wheel_leg_humanoid_lab/wheel_leg_humanoid_lab/assets/utils/get_com_from_urdf.py 	modified:   source/wheel_leg_humanoid_lab/wheel_leg_humanoid_lab/assets/wheel_leg_humanoid_description/urdf/wheel_leg_humanoid.urdf

File: source/wheel_leg_humanoid_lab/wheel_leg_humanoid_lab/assets/wheel_leg_humanoid_description/urdf/wheel_leg_humanoid.urdf (robot description, URDF)
Before this commit: robot wheel_leg_humanoid, 20 links, 19 joints
Links:
- link left_ankle_2: mass 1.55786 -> 1.35786
- link left_foot_wheel_L: mass 0.23598528385264375 -> 0.1
- link left_foot_wheel_R: mass 0.2359852838526443 -> 0.1
- link left_thigh: mass 5.25364 -> 4.25364
- link right_ankle_2: mass 1.55786 -> 1.35786
- link right_foot_wheel_L: mass 0.235985283852645 -> 0.1
- link right_foot_wheel_R: mass 0.235985283852645 -> 0.1
- link right_thigh: mass 5.25364 -> 4.25364
