Commit message: new file:   scripts/eval/checkpoints/driving_flat.pt 	new file:   scripts/eval/checkpoints/driving_rough.pt 	modified:   scripts/eval/checkpoints/walking_flat.pt 	modified:   scripts/eval/inference.py 	renamed:    source/wheel_leg_humanoid_lab/data/Robots/kimm/wheel_leg_humanoid_description/meshes/left_ankle_1.stl -> source/wheel_leg_humanoid_lab/data/Robots/kimm/wheel_leg_humanoid_description/meshes/left_ankle_pitch_link.stl 	renamed:    source/wheel_leg_humanoid_lab/data/Robots/kimm/wheel_leg_humanoid_description/meshes/left_ankle_2.stl -> source/wheel_leg_humanoid_lab/data/Robots/kimm/wheel_leg_humanoid_description/meshes/left_ankle_roll_link.stl 	renamed:    source/wheel_leg_humanoid_lab/data/Robots/kimm/wheel_leg_humanoid_description/meshes/left_foot_wheel_L.stl -> source/wheel_leg_humanoid_lab/data/Robots/kimm/wheel_leg_humanoid_description/meshes/left_foot_wheel_link_L.stl 	renamed:    source/wheel_leg_humanoid_lab/data/Robots/kimm/wheel_leg_humanoid_description/meshes/left_foot_wheel_R.stl -> source/wheel_leg_humanoid_lab/data/Robots/kimm/wheel_leg_humanoid_description/meshes/left_foot_wheel_link_R.stl 	renamed:    source/wheel_leg_humanoid_lab/data/Robots/kimm/wheel_leg_humanoid_description/meshes/left_pelvis_1.stl -> source/wheel_leg_humanoid_lab/data/Robots/kimm/wheel_leg_humanoid_description/meshes/left_hip_pitch_link.stl 	renamed:    source/wheel_leg_humanoid_lab/data/Robots/kimm/wheel_leg_humanoid_description/meshes/left_pelvis_2.stl -> source/wheel_leg_humanoid_lab/data/Robots/kimm/wheel_leg_humanoid_description/meshes/left_hip_roll_link.stl 	renamed:    source/wheel_leg_humanoid_lab/data/Robots/kimm/wheel_leg_humanoid_description/meshes/left_thigh.stl -> source/wheel_leg_humanoid_lab/data/Robots/kimm/wheel_leg_humanoid_description/meshes/left_hip_yaw_link.stl 	renamed:    source/wheel_leg_humanoid_lab/data/Robots/kimm/wheel_leg_humanoid_description/meshes/left_calf.stl -> source/wheel_leg_humanoid_lab/data/Robots/kimm/wheel_leg_humanoid_description/meshes/left_knee_link.stl 	renamed:    source/wheel_leg_humanoid_lab/data/Robots/kimm/wheel_leg_humanoid_description/meshes/left_wheel.stl -> source/wheel_leg_humanoid_lab/data/Robots/kimm/wheel_leg_humanoid_description/meshes/left_wheel_link.stl 	renamed:    source/wheel_leg_humanoid_lab/data/Robots/kimm/wheel_leg_humanoid_description/meshes/waist.stl -> source/wheel_leg_humanoid_lab/data/Robots/kimm/wheel_leg_humanoid_description/meshes/pelvis.stl 	renamed:    source/wheel_leg_humanoid_lab/data/Robots/kimm/wheel_leg_humanoid_description/meshes/right_ankle_1.stl -> source/wheel_leg_humanoid_lab/data/Robots/kimm/wheel_leg_humanoid_description/meshes/right_ankle_pitch_link.stl 	renamed:    source/wheel_leg_humanoid_lab/data/Robots/kimm/wheel_leg_humanoid_description/meshes/right_ankle_2.stl -> source/wheel_leg_humanoid_lab/data/Robots/kimm/wheel_leg_humanoid_description/meshes/right_ankle_roll_link.stl 	renamed:    source/wheel_leg_humanoid_lab/data/Robots/kimm/wheel_leg_humanoid_description/meshes/right_foot_wheel_L.stl -> source/wheel_leg_humanoid_lab/data/Robots/kimm/wheel_leg_humanoid_description/meshes/right_foot_wheel_link_L.stl 	renamed:    source/wheel_leg_humanoid_lab/data/Robots/kimm/wheel_leg_humanoid_description/meshes/right_foot_wheel_R.stl -> source/wheel_leg_humanoid_lab/data/Robots/kimm/wheel_leg_humanoid_description/meshes/right_foot_wheel_link_R.stl 	renamed:    source/wheel_leg_humanoid_lab/data/Robots/kimm/wheel_leg_humanoid_description/meshes/right_pelvis_1.stl -> source/wheel_leg_humanoid_lab/data/Robots/kimm/wheel_leg_humanoid_description/meshes/right_hip_pitch_link.stl 	renamed:    source/wheel_leg_humanoid_lab/data/Robots/kimm/wheel_leg_humanoid_description/meshes/right_pelvis_2.stl -> source/wheel_leg_humanoid_lab/data/Robots/kimm/wheel_leg_humanoid_description/meshes/right_hip_roll_link.stl 	renamed:    source/wheel_leg_humanoid_lab/data/Robots/kimm/wheel_leg_humanoid_description/meshes/right_thigh.stl -> source/wheel_leg_humanoid_lab/data/Robots/kimm/wheel_leg_humanoid_description/meshes/right_hip_yaw_link.stl 	renamed:    source/wheel_leg_humanoid_lab/data/Robots/kimm/wheel_leg_humanoid_description/meshes/right_calf.stl -> source/wheel_leg_humanoid_lab/data/Robots/kimm/wheel_leg_humanoid_description/meshes/right_knee_link.stl 	renamed:    source/wheel_leg_humanoid_lab/data/Robots/kimm/wheel_leg_humanoid_description/meshes/right_wheel.stl -> source/wheel_leg_humanoid_lab/data/Robots/kimm/wheel_leg_humanoid_description/meshes/right_wheel_link.stl 	renamed:    source/wheel_leg_humanoid_lab/data/Robots/kimm/wheel_leg_humanoid_description/meshes/base_link.stl -> source/wheel_leg_humanoid_lab/data/Robots/kimm/wheel_leg_humanoid_description/meshes/torso_link.stl 	modified:   source/wheel_leg_humanoid_lab/data/Robots/kimm/wheel_leg_humanoid_description/urdf/wheel_leg_humanoid.urdf 	new file:   source/wheel_leg_humanoid_lab/data/Robots/kimm/wheel_leg_humanoid_description/urdf/wheel_leg_humanoid/configuration/wheel_leg_humanoid_base.usd 	new file:   source/wheel_leg_humanoid_lab/data/Robots/kimm/wheel_leg_humanoid_description/urdf/wheel_leg_humanoid/configuration/wheel_leg_humanoid_physics.usd 	new file:   source/wheel_leg_humanoid_lab/data/Robots/kimm/wheel_leg_humanoid_description/urdf/wheel_leg_humanoid/configuration/wheel_leg_humanoid_robot.usd 	new file:   source/wheel_leg_humanoid_lab/data/Robots/kimm/wheel_leg_humanoid_description/urdf/wheel_leg_humanoid/configuration/wheel_leg_humanoid_sensor.usd 	new file:   source/wheel_leg_humanoid_lab/data/Robots/kimm/wheel_leg_humanoid_description/urdf/wheel_leg_humanoid/wheel_leg_humanoid.usd 	modified:   source/wheel_leg_humanoid_lab/wheel_leg_humanoid_lab/assets/robot/utils/get_com_from_urdf.py 	modified:   source/wheel_leg_humanoid_lab/wheel_leg_humanoid_lab/assets/robot/wheel_leg_humanoid.py 	modified:   source/wheel_leg_humanoid_lab/wheel_leg_humanoid_lab/tasks/manager_based/wheel_leg_humanoid/velocity/config/drving/rough_env_cfg.py 	modified:   source/wheel_leg_humanoid_lab/wheel_leg_humanoid_lab/tasks/manager_based/wheel_leg_humanoid/velocity/config/walking/flat_env_cfg.py 	modified:   source/wheel_leg_humanoid_lab/wheel_leg_humanoid_lab/tasks/manager_based/wheel_leg_humanoid/velocity/config/walking/rough_env_cfg.py

File: source/wheel_leg_humanoid_lab/data/Robots/kimm/wheel_leg_humanoid_description/urdf/wheel_leg_humanoid.urdf (robot description, URDF)
Before this commit: robot wheel_leg_humanoid, 20 links, 19 joints
Links:
- removed link base_link
- removed link left_ankle_1
- removed link left_ankle_2
- removed link left_calf
- removed link left_foot_wheel_L
- removed link left_foot_wheel_R
- removed link left_pelvis_1
- removed link left_pelvis_2
- removed link left_thigh
- removed link left_wheel
- removed link right_ankle_1
- removed link right_ankle_2
- removed link right_calf
- removed link right_foot_wheel_L
- removed link right_foot_wheel_R
- removed link right_pelvis_1
- removed link right_pelvis_2
- removed link right_thigh
- removed link right_wheel
- removed link waist
- added link base; visual box size=0.001 0.001 0.001
- added link left_ankle_pitch_link, mass 0.26578; collision mesh filename=package://wheel_leg_humanoid_description/meshes/left_ankle_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 scale=0.001 0.001 0.001; visual mesh filename=package://wheel_leg_humanoid_description/meshes/left_ankle_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 scale=0.001 0.001 0.001
- added link left_ankle_roll_link, mass 1.35786; collision mesh filename=package://wheel_leg_humanoid_description/meshes/left_ankle_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 scale=0.001 0.001 0.001; visual mesh filename=package://wheel_leg_humanoid_description/meshes/left_ankle_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 scale=0.001 0.001 0.001
- added link left_foot_wheel_link_L, mass 0.1; collision mesh filename=package://wheel_leg_humanoid_description/meshes/left_foot_w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 scale=0.001 0.001 0.001; visual mesh filename=package://wheel_leg_humanoid_description/meshes/left_foot_w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 scale=0.001 0.001 0.001
- added link left_foot_wheel_link_R, mass 0.1; collision mesh filename=package://wheel_leg_humanoid_description/meshes/left_foot_w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 scale=0.001 0.001 0.001; visual mesh filename=package://wheel_leg_humanoid_description/meshes/left_foot_w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 scale=0.001 0.001 0.001
- added link left_hip_pitch_link, mass 1.32134; collision mesh filename=package://wheel_leg_humanoid_description/meshes/left_hip_pi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 scale=0.001 0.001 0.001; visual mesh filename=package://wheel_leg_humanoid_description/meshes/left_hip_pi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 scale=0.001 0.001 0.001
- added link left_hip_roll_link, mass 1.24911; collision mesh filename=package://wheel_leg_humanoid_description/meshes/left_hip_ro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 scale=0.001 0.001 0.001; visual mesh filename=package://wheel_leg_humanoid_description/meshes/left_hip_ro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 scale=0.001 0.001 0.001
- added link left_hip_yaw_link, mass 4.25364; collision mesh filename=package://wheel_leg_humanoid_description/meshes/left_hip_ya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 scale=0.001 0.001 0.001; visual mesh filename=package://wheel_leg_humanoid_description/meshes/left_hip_ya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 scale=0.001 0.001 0.001
- added link left_knee_link, mass 1.88334; collision mesh filename=package://wheel_leg_humanoid_description/meshes/left_knee_l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 scale=0.001 0.001 0.001; visual mesh filename=package://wheel_leg_humanoid_description/meshes/left_knee_l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 scale=0.001 0.001 0.001
- added link left_wheel_link, mass 1.0; collision mesh filename=package://wheel_leg_humanoid_description/meshes/left_wheel_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 scale=0.001 0.001 0.001; visual mesh filename=package://wheel_leg_humanoid_description/meshes/left_wheel_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 scale=0.001 0.001 0.001
- added link pelvis, mass 2.7388; collision mesh filename=package://wheel_leg_humanoid_description/meshes/pelvis.stl scale=0.001 0.001 0.001; visual mesh filename=package://wheel_leg_humanoid_description/meshes/pelvis.stl scale=0.001 0.001 0.001
- added link right_ankle_pitch_link, mass 0.26578; collision mesh filename=package://wheel_leg_humanoid_description/meshes/right_ankle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 scale=0.001 0.001 0.001; visual mesh filename=package://wheel_leg_humanoid_description/meshes/right_ankle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 scale=0.001 0.001 0.001
- added link right_ankle_roll_link, mass 1.35786; collision mesh filename=package://wheel_leg_humanoid_description/meshes/right_ankle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 scale=0.001 0.001 0.001; visual mesh filename=package://wheel_leg_humanoid_description/meshes/right_ankle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 scale=0.001 0.001 0.001
- added link right_foot_wheel_link_L, mass 0.1; collision mesh filename=package://wheel_leg_humanoid_description/meshes/right_foot_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 scale=0.001 0.001 0.001; visual mesh filename=package://wheel_leg_humanoid_description/meshes/right_foot_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 scale=0.001 0.001 0.001
- added link right_foot_wheel_link_R, mass 0.1; collision mesh filename=package://wheel_leg_humanoid_description/meshes/right_foot_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 scale=0.001 0.001 0.001; visual mesh filename=package://wheel_leg_humanoid_description/meshes/right_foot_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 scale=0.001 0.001 0.001
- added link right_hip_pitch_link, mass 1.32134; collision mesh filename=package://wheel_leg_humanoid_description/meshes/right_hip_p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 scale=0.001 0.001 0.001; visual mesh filename=package://wheel_leg_humanoid_description/meshes/right_hip_p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 scale=0.001 0.001 0.001
- added link right_hip_roll_link, mass 1.24911; collision mesh filename=package://wheel_leg_humanoid_description/meshes/right_hip_r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 scale=0.001 0.001 0.001; visual mesh filename=package://wheel_leg_humanoid_description/meshes/right_hip_r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 scale=0.001 0.001 0.001
- added link right_hip_yaw_link, mass 4.25364; collision mesh filename=package://wheel_leg_humanoid_description/meshes/right_hip_y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 scale=0.001 0.001 0.001; visual mesh filename=package://wheel_leg_humanoid_description/meshes/right_hip_y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 scale=0.001 0.001 0.001
- added link right_knee_link, mass 1.88334; collision mesh filename=package://wheel_leg_humanoid_description/meshes/right_knee_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 scale=0.001 0.001 0.001; visual mesh filename=package://wheel_leg_humanoid_description/meshes/right_knee_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 scale=0.001 0.001 0.001
- added link right_wheel_link, mass 1.0; collision mesh filename=package://wheel_leg_humanoid_description/meshes/right_wheel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 scale=0.001 0.001 0.001; visual mesh filename=package://wheel_leg_humanoid_description/meshes/right_wheel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 scale=0.001 0.001 0.001
- added link torso_link, mass 12.883; collision mesh filename=package://wheel_leg_humanoid_description/meshes/torso_link.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 scale=0.001 0.001 0.001; visual mesh filename=package://wheel_leg_humanoid_description/meshes/torso_link.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 scale=0.001 0.001 0.001
Joints:
- removed joint left_ankle_1
- removed joint left_ankle_2
- removed joint left_calf
- removed joint left_foot_wheel_L
- removed joint left_foot_wheel_R
- removed joint left_pelvis_1
- removed joint left_pelvis_2
- removed joint left_thigh
- removed joint left_wheel
- removed joint right_ankle_1
- removed joint right_ankle_2
- removed joint right_calf
- removed joint right_foot_wheel_L
- removed joint right_foot_wheel_R
- removed joint right_pelvis_1
- removed joint right_pelvis_2
- removed joint right_thigh
- removed joint right_wheel
- removed joint waist
- added joint floating_base: type fixed, parent base, child pelvis, origin xyz=0 0 0 rpy=0 0 0
- added joint left_ankle_pitch_joint: type revolute, parent left_knee_link, child left_ankle_pitch_link, origin xyz=5e-05 -0.03575 -0.34005 rpy=0 0 0, axis 0.0 1.0 -0.0, limit lower=-0.87 upper=0.52 effort=120 velocity=5.02
- added joint left_ankle_roll_joint: type revolute, parent left_ankle_pitch_link, child left_ankle_roll_link, origin xyz=0.0335 -0.0035 -0.042 rpy=0 0 0, axis 1.0 0.0 0.0, limit lower=-0.26 upper=0.26 effort=120 velocity=5.02
- added joint left_foot_wheel_joint_L: type continuous, parent left_ankle_roll_link, child left_foot_wheel_link_L, origin xyz=0.121425 0.054649 -0.000937 rpy=0 0 0, axis 0.0 1.0 0.0
- added joint left_foot_wheel_joint_R: type continuous, parent left_ankle_roll_link, child left_foot_wheel_link_R, origin xyz=0.121425 -0.054851 -0.000762 rpy=0 0 0, axis 0.0 1.0 -0.000799
- added joint left_hip_pitch_joint: type revolute, parent pelvis, child left_hip_pitch_link, origin xyz=0.0 0.06325 0 rpy=0 0 0, axis 0.0 1.0 0.0, limit lower=-2.53 upper=2.88 effort=120 velocity=5.02
- added joint left_hip_roll_joint: type revolute, parent left_hip_pitch_link, child left_hip_roll_link, origin xyz=0.03625 0.07915 0.0 rpy=0 0 0, axis 1.0 -0.0 0.0, limit lower=-0.52 upper=2.97 effort=120 velocity=5.02
- added joint left_hip_yaw_joint: type revolute, parent left_hip_roll_link, child left_hip_yaw_link, origin xyz=-0.03635 0.0 -0.11575 rpy=0 0 0, axis 0.0 0.0 1.0, limit lower=-2.76 upper=2.76 effort=120 velocity=5.02
- added joint left_knee_joint: type revolute, parent left_hip_yaw_link, child left_knee_link, origin xyz=0.0 0.03925 -0.23415 rpy=0 0 0, axis 0.0 1.0 -0.0, limit lower=-0.087 upper=2.88 effort=120 velocity=5.02
- added joint left_wheel_joint: type continuous, parent left_hip_yaw_link, child left_wheel_link, origin xyz=5e-05 0.07905 -0.2342 rpy=0 0 0, axis 0.0 1.0 -0.0, limit effort=120 velocity=5.02
- added joint right_ankle_pitch_joint: type revolute, parent right_knee_link, child right_ankle_pitch_link, origin xyz=-0.00045 0.03575 -0.34005 rpy=0 0 0, axis 0.0 1.0 0.0, limit lower=-0.87 upper=0.52 effort=120 velocity=5.02
- added joint right_ankle_roll_joint: type revolute, parent right_ankle_pitch_link, child right_ankle_roll_link, origin xyz=0.0335 0.0035 -0.042 rpy=0 0 0, axis 1.0 0.0 0.0, limit lower=-0.26 upper=0.26 effort=120 velocity=5.02
- added joint right_foot_wheel_joint_L: type continuous, parent right_ankle_roll_link, child right_foot_wheel_link_L, origin xyz=0.121925 0.054845 -0.001102 rpy=0 0 0, axis 0.0 1.0 0.0
- added joint right_foot_wheel_joint_R: type continuous, parent right_ankle_roll_link, child right_foot_wheel_link_R, origin xyz=0.121925 -0.054653 -0.000598 rpy=0 0 0, axis 0.0 0.999997 -0.002304
- added joint right_hip_pitch_joint: type revolute, parent pelvis, child right_hip_pitch_link, origin xyz=0.0 -0.06325 0 rpy=0 0 0, axis 0.0 1.0 0.0, limit lower=-2.53 upper=2.88 effort=120 velocity=5.02
- added joint right_hip_roll_joint: type revolute, parent right_hip_pitch_link, child right_hip_roll_link, origin xyz=0.03875 -0.07915 0.0 rpy=0 0 0, axis 1.0 -0.0 0.0, limit lower=-2.97 upper=0.52 effort=120 velocity=5.02
- added joint right_hip_yaw_joint: type revolute, parent right_hip_roll_link, child right_hip_yaw_link, origin xyz=-0.03785 0.0 -0.11575 rpy=0 0 0, axis 0.0 0.0 1.0, limit lower=-2.76 upper=2.76 effort=120 velocity=5.02
- added joint right_knee_joint: type revolute, parent right_hip_yaw_link, child right_knee_link, origin xyz=0.0 -0.03925 -0.23415 rpy=0 0 0, axis 0.0 1.0 0.0, limit lower=-0.087 upper=2.88 effort=120 velocity=5.02
- added joint right_wheel_joint: type continuous, parent right_hip_yaw_link, child right_wheel_link, origin xyz=-0.00045 -0.07905 -0.2342 rpy=0 0 0, axis 0.0 1.0 0.0, limit effort=120 velocity=5.02
- added joint waist_yaw_joint: type revolute, parent pelvis, child torso_link, origin xyz=0.0 0.0 0.0862 rpy=0 0 0, axis -0.0 0.0 1.0, limit lower=-2.62 upper=2.62 effort=120 velocity=5.02
